Commit message: Updating lidar urdf to find meshes via file location

File: velodyne_description/urdf/HDL-32E.urdf.xacro (robot description, xacro)
@@ -18,5 +18,5 @@
       <visual>
         <geometry>
-          <mesh filename="package://velodyne_description/meshes/HDL32E_base.dae" />
+          <mesh filename="file://$(find velodyne_description)/meshes/HDL32E_base.dae" />
         </geometry>
       </visual>
@@ -42,5 +42,5 @@
         <origin xyz="0 0 -0.09081" rpy="0 0 0" />
         <geometry>
-          <mesh filename="package://velodyne_description/meshes/HDL32E_scan.dae" />
+          <mesh filename="file://$(find velodyne_description)/meshes/HDL32E_scan.dae" />
         </geometry>
       </visual>
@@ -79,5 +79,5 @@
             </noise>
           </ray>
-          <plugin name="gazebo_ros_laser_controller" filename="libgazebo_ros_velodyne_laser.so">
+          <plugin name="gazebo_ros_laser_controller" filename="./libgazebo_ros_velodyne_laser.so">
             <topicName>${topic}</topicName>
             <frameName>${name}</frameName>
@@ -119,5 +119,5 @@
             </noise>
           </ray>
-          <plugin name="gazebo_ros_laser_controller" filename="libgazebo_ros_velodyne_laser.so">
+          <plugin name="gazebo_ros_laser_controller" filename="./libgazebo_ros_velodyne_laser.so">
             <topicName>${topic}</topicName>
             <frameName>${name}</frameName>

File: velodyne_description/urdf/VLP-16.urdf.xacro (robot description, xacro)
@@ -16,10 +16,10 @@
       <visual>
         <geometry>
-          <mesh filename="package://velodyne_description/meshes/VLP16_base_1.dae"/>
+          <mesh filename="file://$(find velodyne_description)/meshes/VLP16_base_1.dae"/>
         </geometry>
       </visual>
       <visual>
         <geometry>
-          <mesh filename="package://velodyne_description/meshes/VLP16_base_2.dae"/>
+          <mesh filename="file://$(find velodyne_description)/meshes/VLP16_base_2.dae"/>
         </geometry>
       </visual>
@@ -45,5 +45,5 @@
         <origin xyz="0 0 -0.0377"/>
         <geometry>
-          <mesh filename="package://velodyne_description/meshes/VLP16_scan.dae"/>
+          <mesh filename="file://$(find velodyne_description)/meshes/VLP16_scan.dae"/>
         </geometry>
       </visual>
@@ -83,5 +83,5 @@
             </noise>
           </ray>
-          <plugin name="gazebo_ros_laser_controller" filename="libgazebo_ros_velodyne_laser.so">
+          <plugin name="gazebo_ros_laser_controller" filename="./libgazebo_ros_velodyne_laser.so">
             <topicName>${topic}</topicName>
             <frameName>${name}</frameName>
@@ -124,5 +124,5 @@
             </noise>
           </ray>
-          <plugin name="gazebo_ros_laser_controller" filename="libgazebo_ros_velodyne_laser.so">
+          <plugin name="gazebo_ros_laser_controller" filename="./libgazebo_ros_velodyne_laser.so">
             <topicName>${topic}</topicName>
             <frameName>${name}</frameName>

File: velodyne_description/urdf/VLP-32C.urdf.xacro (robot description, xacro)
@@ -17,10 +17,10 @@
       <visual>
         <geometry>
-          <mesh filename="package://velodyne_description/meshes/VLP16_base_1.dae"/>
+          <mesh filename="file://$(find velodyne_description)/meshes/VLP16_base_1.dae"/>
         </geometry>
       </visual>
       <visual>
         <geometry>
-          <mesh filename="package://velodyne_description/meshes/VLP16_base_2.dae"/>
+          <mesh filename="file://$(find velodyne_description)/meshes/VLP16_base_2.dae"/>
         </geometry>
       </visual>
@@ -46,5 +46,5 @@
         <origin xyz="0 0 -0.0377"/>
         <geometry>
-          <mesh filename="package://velodyne_description/meshes/VLP16_scan.dae"/>
+          <mesh filename="file://$(find velodyne_description)/velodyne_description/meshes/VLP16_scan.dae"/>
         </geometry>
       </visual>
@@ -83,5 +83,5 @@
             </noise>
           </ray>
-          <plugin name="gazebo_ros_laser_controller" filename="libgazebo_ros_velodyne_laser.so">
+          <plugin name="gazebo_ros_laser_controller" filename="./libgazebo_ros_velodyne_laser.so">
             <topicName>${topic}</topicName>
             <frameName>${name}</frameName>
@@ -137,5 +137,5 @@
             </noise>
           </ray>
-          <plugin name="gazebo_ros_laser_controller" filename="libgazebo_ros_velodyne_laser.so">
+          <plugin name="gazebo_ros_laser_controller" filename="./libgazebo_ros_velodyne_laser.so">
             <topicName>${topic}</topicName>
             <frameName>${name}</frameName>
